Commit message: finally, a working configuration -- let it never be touched.

File: urdf/udacity_bot.xacro (robot description, xacro)
@@ -2,6 +2,6 @@
 <robot name="udacity_bot" xmlns:xacro="http://ros.org/wiki/xacro">
     <xacro:include filename="$(find udacity_bot)/urdf/common.xacro"/>
+    <link name="robot_footprint"></link>
     <xacro:include filename="$(find udacity_bot)/urdf/udacity_bot.gazebo"/>
-    <link name="robot_footprint"></link>
     <joint name="robot_footprint_joint" type="fixed">
         <origin xyz="0 0 0" rpy="0 0 0" />

Commit message: add visualizations and evaluation scripts, as well as a more convenient navigation_goal.cpp

File: urdf/udacity_bot.xacro (robot description, xacro)
@@ -105,5 +105,5 @@
         <parent link="chassis"/>
         <child link="laser"/>
-        <origin xyz="0.15 0 0.1" rpy="0 0 0"/>
+        <origin xyz="0.0 0 0.1" rpy="0 0 0"/>
     </joint>
 </robot>
