Commit message: re-tuning contact params for udacity_bot

File: urdf/common.xacro (robot description, xacro)
@@ -31,5 +31,5 @@
 			</inertial>
 			<visual>
-				<origin xyz="0 0 0" rpy="${pi/2} 0 0"/>
+				<origin xyz="0 0 0" rpy="0 0 0"/>
 				<geometry>
 					<cylinder length="${wheel_thickness}" radius="${wheel_radius}"/>
@@ -40,5 +40,6 @@
 			</visual>
 			<collision>
-				<origin xyz="0.0 0.0 0" rpy="${pi/2} 0 0"/>
+				<self_collide>false</self_collide>
+				<origin xyz="0.0 0.0 0" rpy="0 0 0"/>
 				<geometry>
 					<cylinder length="${wheel_thickness}" radius="${wheel_radius}"/>
@@ -51,5 +52,5 @@
 			<xacro:insert_block name="origin"/>
 			<!---<joint_properties damping="0.0" friction="0.5"/>-->
-			<axis xyz="0 1 0" rpy="0 0 0"/>
+			<axis xyz="0 0 1"/>
 			<limit effort="10000" velocity="1000"/>
 			<dynamics damping="1.0" friction="1.0"/>

File: urdf/udacity_bot.xacro (robot description, xacro)
@@ -1,65 +1,69 @@
 <?xml version='1.0'?>
 <robot name="udacity_bot" xmlns:xacro="http://ros.org/wiki/xacro">
+	<!-- body -->
+	<xacro:property name="br" value="0.25"/>
+	<xacro:property name="bh" value="0.1"/>
+	<!-- wheel -->
+	<xacro:property name="wr" value="0.05"/>
+	<xacro:property name="wd" value="0.3"/>
+	<xacro:property name="wt" value="0.01"/>
+	<!-- caster -->
+	<xacro:property name="cr" value="0.04"/>
     <xacro:include filename="$(find udacity_bot)/urdf/common.xacro"/>
+    <xacro:include filename="$(find udacity_bot)/urdf/udacity_bot.gazebo"/>
     <link name="robot_footprint"></link>
-    <xacro:include filename="$(find udacity_bot)/urdf/udacity_bot.gazebo"/>
     <joint name="robot_footprint_joint" type="fixed">
-        <origin xyz="0 0 0" rpy="0 0 0" />
+		<origin xyz="0 0 ${wr}" rpy="0 0 0" />
         <parent link="robot_footprint"/>
         <child link="chassis" />
     </joint>
     <link name='chassis'>
-        <pose>0 0 0.1 0 0 0</pose>
         <inertial>
             <mass value="15.0"/>
-            <origin xyz="0.0 0 0" rpy=" 0 0 0"/>
-            <inertia
-                ixx="0.1" ixy="0" ixz="0"
-                iyy="0.1" iyz="0"
-                izz="0.1"
-                />
+			<origin xyz="0 0 ${wr}" rpy="0 0 0"/>
+			<cylinder_inertia m="15" r="${br}" h="${bh}"/>
         </inertial>
         <collision name='collision'>
-            <origin xyz="0 0 0" rpy=" 0 0 0"/>
+			<origin xyz="0 0 ${wr}" rpy="0 0 0"/>
             <geometry>
-                <box size=".4 .2 .1"/>
+				<cylinder length="${bh}" radius="${br}"/>
             </geometry>
         </collision>
         <visual name='chassis_visual'>
-            <origin xyz="0 0 0" rpy=" 0 0 0"/>
+			<origin xyz="0 0 ${wr}" rpy="0 0 0"/>
             <geometry>
-                <box size=".4 .2 .1"/>
+				<cylinder length="${bh}" radius="${br}"/>
             </geometry>
         </visual>
         <collision name='back_caster_collision'>
-            <origin xyz="-0.15 0 -0.05" rpy=" 0 0 0"/>
+			<origin xyz="-0.15 0 ${-wr+cr}" rpy=" 0 0 0"/>
             <geometry>
-                <sphere radius="0.0499"/>
+				<sphere radius="${cr}"/>
             </geometry>
         </collision>
         <visual name='back_caster_visual'>
-            <origin xyz="-0.15 0 -0.05" rpy=" 0 0 0"/>
+			<origin xyz="-0.15 0 ${-wr+cr}" rpy=" 0 0 0"/>
             <geometry>
-                <sphere radius="0.05"/>
+				<sphere radius="${cr}"/>
             </geometry>
         </visual>
         <collision name='front_caster_collision'>
-            <origin xyz="0.15 0 -0.05" rpy=" 0 0 0"/>
+			<origin xyz="0.15 0 ${-wr+cr}" rpy=" 0 0 0"/>
             <geometry>
-                <sphere radius="0.0499"/>
+				<sphere radius="${cr}"/>
             </geometry>
         </collision>
         <visual name='front_caster_visual'>
-            <origin xyz="0.15 0 -0.05" rpy=" 0 0 0"/>
+			<origin xyz="0.15 0 ${-wr+cr}" rpy=" 0 0 0"/>
             <geometry>
-                <sphere radius="0.05"/>
+				<sphere radius="${cr}"/>
             </geometry>
         </visual>
     </link>
-    <xacro:wheel wheel_prefix="left" wheel_mass="5" wheel_radius="0.1" wheel_thickness="0.05" parent="chassis">
-        <origin xyz="0 0.15 0" rpy="0 0 0"/>
+	<xacro:wheel wheel_prefix="left" wheel_mass="5" wheel_radius="${wr}" wheel_thickness="${wt}" parent="chassis">
+		<origin xyz="0 ${wd/2} 0" rpy="${-pi/2} 0 0"/>
     </xacro:wheel>
-    <xacro:wheel wheel_prefix="right" wheel_mass="5" wheel_radius="0.1" wheel_thickness="0.05" parent="chassis">
-        <origin xyz="0 -0.15 0" rpy="0 0 0"/>
+	<xacro:wheel wheel_prefix="right" wheel_mass="5" wheel_radius="${wr}" wheel_thickness="${wt}" parent="chassis">
+		<origin xyz="0 ${-wd/2} 0" rpy="${-pi/2} 0 0"/>
     </xacro:wheel>
     <link name="camera">
@@ -84,5 +88,5 @@
         <parent link="chassis"/>
         <child link="camera"/>
-        <origin xyz="0.2 0 0" rpy="0 0 0"/>
+        <origin xyz="0.25 0 0.05" rpy="0 0 0"/>
     </joint>
     <link name="laser">
